File: BLDC_driver/BLDC_driver.kicad_pcb (KiCad board)
At the start: 4 copper layers, 100 x 100 mm, 125 parts, among them J1 CTRL, J2 POWER, J3 JTAG, J4 USB-C 16P, Q1 AOTL66912, Q10 AOTL66912, Q11 AOTL66912, Q12 AOTL66912, Q13 AOTL66912, Q14 AOTL66912, Q15 AOTL66912, Q16 AOTL66912, Q17 AOTL66912, Q18 AOTL66912, Q2 AOTL66912, Q3 AOTL66912, Q4 AOTL66912, Q5 AOTL66912, Q6 AOTL66912, Q7 AOTL66912, Q8 AOTL66912, Q9 AOTL66912, SW1 BTN, SW2 BTN, U1 STM32F412CEUx, U2 W25Q128JVS, U3 USBLC6-2SC6, Y1 25MHz

Commit message: Layout progress
Parts:
- removed H1, H2, H3, H4: MountingHole_Pad, MountingHole:MountingHole_3.2mm_M3_Pad_Via
- added C5: 2u2/100v, Capacitor_SMD:C_1210_3225Metric, F.Cu at (76.2, 82.0)
- added C6: 2u2/100v, Capacitor_SMD:C_1210_3225Metric, F.Cu at (76.2, 105.4)
- added C7: 2u2/100v, Capacitor_SMD:C_1210_3225Metric, F.Cu at (76.2, 128.7)
- added C8: 2u2/100v, Capacitor_SMD:C_1210_3225Metric, F.Cu at (76.2, 152.0)
- C19: renamed from C15; moved to B.Cu
- D3, D6, D9, R16, R34: moved to B.Cu
- moved J4 115.2 mm to (162.3, 112.0), turned to 90 degrees
- moved R6 111.5 mm to (172.5, 112.6), turned to 90 degrees
- moved FL1 109.8 mm to (170.1, 112.6), turned to 90 degrees
- moved U3 98.0 mm to (176.5, 112.8), turned to 180 degrees
- moved D2 79.8 mm to (191.7, 140.7)
- moved C10 79.8 mm to (173.8, 126.0)
- moved C11 79.8 mm to (173.8, 128.5)
- moved C12 79.8 mm to (173.8, 131.0)
- moved C13 79.8 mm to (173.8, 133.5)
- moved C14 79.8 mm to (177.8, 123.5)
- moved C15 79.8 mm to (177.8, 126.0)
- moved C16 79.8 mm to (177.8, 128.5)
- moved C17 79.8 mm to (177.8, 131.0)
- moved C9 79.8 mm to (173.8, 123.5)
- moved D1 79.8 mm to (191.7, 138.1)
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- renumbered C6 to C10, C7 to C11, C8 to C12, C9 to C13, C10 to C14, C11 to C15, C12 to C16, C13 to C17, C14 to C18, C16 to C20, C17 to C21, C18 to C22, C19 to C23, C20 to C24, C21 to C25, C22 to C26, C23 to C27, C24 to C28, C25 to C29, C26 to C30, C27 to C31, C28 to C32, C29 to C33, C30 to C34, C31 to C35, C32 to C36, C33 to C37, C34 to C38, C35 to C39, C36 to C40, C37 to C41, C5 to C9
Routing:
- net /inverter stage/HA: track 85.1 -> 99.5 mm, vias 0 -> 1
- net GND: track 6.39 -> 18.9 mm, vias 0 -> 150
- net /inverter stage/PHB: track 0.00 -> 11.1 mm, vias 0 -> 1
- net /inverter stage/PHA: track 0.00 -> 6.69 mm, vias 0 -> 1
- net /inverter stage/LSA: track 0.00 -> 5.00 mm
- net +12V: track 2.36 -> 7.08 mm
- net /inverter stage/HSA: track 0.00 -> 4.63 mm
- net /inverter stage/LSB: track 1.60 -> 5.00 mm
- net /inverter stage/LSC: track 1.60 -> 4.87 mm
- net /inverter stage/HSB: track 1.60 -> 4.61 mm
- net /inverter stage/A: track 18.0 -> 20.9 mm
- net Net-(U5-HB): track 0.00 -> 2.82 mm, vias 0 -> 1
- net /inverter stage/LA: track 37.7 -> 40.6 mm, vias 6 -> 7
- net Net-(D3-K): track 0.00 -> 1.24 mm, vias 0 -> 1
- net Net-(D6-K): track 0.00 -> 1.23 mm, vias 0 -> 1
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