File: BLDC_driver/inverter_stage.kicad_sch (KiCad schematic)
At the start: 66 parts, among them Q1 AOTL66912, Q2 AOTL66912, Q3 AOTL66912, Q4 AOTL66912, Q5 AOTL66912, Q6 AOTL66912

Commit message: New design
Parts:
- removed C10, C11, C12, C13, C14, C15: 3.3nF, Capacitor_SMD:C_0805_2012Metric, symbol Device:C_Small
- removed Q1, Q2, Q3, Q4, Q5, Q6: AOTL66912, Package_TO_SOT_SMD:Infineon_PG-HSOF-8-1_ThermalVias, symbol Marijn:AOTL66912
- removed R10, R11, R12, R7, R8, R9: 2R2, Resistor_SMD:R_0603_1608Metric, symbol Device:R_Small
- renumbered C19 to C14, C16 to C15, C20 to C16, C21 to C18, C18 to C19, D4 to D10, D5 to D11, D6 to D3, D8 to D4, D9 to D5, D7 to D6, D10 to D7, D11 to D8, D3 to D9, R20 to R10, R27 to R11, R30 to R12, R21 to R13, R28 to R14, R31 to R15, R22 to R16, R38 to R17, R39 to R18, R23 to R19, R32 to R20, R35 to R21, R24 to R22, R33 to R23, R36 to R24, R13 to R25, R14 to R26, R15 to R27, R25 to R28, R34 to R29, R37 to R30, R16 to R31, R17 to R32, R18 to R33, R19 to R7, R26 to R8, R29 to R9
Connections:
- net HA: now reaches D3.2 (A), R10.2, R13.2
- net LB: now reaches D7.2 (A), R23.2, R29.2
- net LA: now reaches D6.2 (A), R22.2, R28.2
- net LC: now reaches D8.2 (A), R24.2, R30.2
- net HC: now reaches D5.2 (A), R12.2, R15.2
- net HB: now reaches D4.2 (A), R11.2, R14.2
Other:
- added sheet gate (gate.kicad_sch)
- added sheet gate1 (gate.kicad_sch)
- added sheet gate2 (gate.kicad_sch)
- added sheet gate3 (gate.kicad_sch)
- added sheet gate4 (gate.kicad_sch)
- added sheet gate5 (gate.kicad_sch)
- note added: "Bridge logic (High current, High voltage, Heat)"
- note added: "Gate driver logic"
- note added: "Gate drivers"
- note removed: "360A max?"
- moved on the sheet: C14, C15, C16, C17, C18, C19, D10, D11, D3, D4, D5, D6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

Commit message: Layout progress
Parts:
- added R26, R28, R30: 500u, Marijn_KiCad:CSS2H-3920R-xxxx, symbol Marijn:CSS2H-3920R-L500F
- R25: value 200u -> 500u
- R27: renamed from R26; value 200u -> 500u
- R29: renamed from R27; value 200u -> 500u
- renumbered R28 to R31, R29 to R32, R30 to R33, R31 to R34, R32 to R35, R33 to R36
Connections:
- net A_CSP: now also R26.1
- net B_CSP: now also R28.1
- net C_CSP: now also R30.1
- net GND: now also R26.2, R28.2, R30.2
Other:
- moved on the sheet: R25, R27, R29

Commit message: Layout progress
Parts:
- renumbered C14 to C18, C15 to C19, C16 to C20, C17 to C21, C18 to C22, C19 to C23
Changed lines of the file:
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@@
 		(on_board yes)
 		(dnp no)
-		(property "Reference" "#PWR031"
+		(property "Reference" "#PWR030"
 			(at 217.17 93.98 0)
 			(effects
@@
 			(project "BLDC_driver"
 				(path "/6f399879-dc45-4210-87b6-ea005f89c132/156cc71e-604a-4062-8209-9f4827fd9816"
-					(reference "#PWR031")
+					(reference "#PWR030")
 					(unit 1)
 				)
@@
 		(dnp no)
 		(fields_autoplaced yes)
-		(property "Reference" "#PWR042"
+		(property "Reference" "#PWR041"
 			(at 86.36 173.99 0)
 			(effects
@@
 			(project "BLDC_driver"
 				(path "/6f399879-dc45-4210-87b6-ea005f89c132/156cc71e-604a-4062-8209-9f4827fd9816"
-					(reference "#PWR042")
+					(reference "#PWR041")
 					(unit 1)
 				)
@@
 		(on_board yes)
 		(dnp no)
-		(property "Reference" "C19"
+		(property "Reference" "C23"
 			(at 76.708 163.83 0)
 			(effects
@@
 			(project "BLDC_driver"
 				(path "/6f399879-dc45-4210-87b6-ea005f89c132/156cc71e-604a-4062-8209-9f4827fd9816"
-					(reference "C19")
+					(reference "C23")
 					(unit 1)
 				)
@@
 		(on_board yes)
 		(dnp no)
-		(property "Reference" "#PWR043"
+		(property "Reference" "#PWR042"
 			(at 45.72 175.26 0)
 			(effects
@@
 			(project "BLDC_driver"
 				(path "/6f399879-dc45-4210-87b6-ea005f89c132/156cc71e-604a-4062-8209-9f4827fd9816"
-					(reference "#PWR043")
+					(reference "#PWR042")
 					(unit 1)
 				)
@@
 		(on_board yes)
 		(dnp no)
-		(property "Reference" "C14"
+		(property "Reference" "C18"
 			(at 41.148 121.158 0)
 			(effects
@@
 			(project "BLDC_driver"
 				(path "/6f399879-dc45-4210-87b6-ea005f89c132/156cc71e-604a-4062-8209-9f4827fd9816"
-					(reference "C14")
+					(reference "C18")
 					(unit 1)
 				)
@@
 		(on_board yes)
 		(dnp no)
-		(property "Reference" "#PWR033"
+		(property "Reference" "#PWR032"
 			(at 74.93 95.25 0)
 			(effects
@@
 			(project "BLDC_driver"
 				(path "/6f399879-dc45-4210-87b6-ea005f89c132/156cc71e-604a-4062-8209-9f4827fd9816"
-					(reference "#PWR033")
+					(reference "#PWR032")
 					(unit 1)
 				)
@@
 		(on_board yes)
 		(dnp no)
-		(property "Reference" "#PWR034"
+		(property "Reference" "#PWR033"
 			(at 100.33 95.25 0)
 			(effects
@@
 			(project "BLDC_driver"
 				(path "/6f399879-dc45-4210-87b6-ea005f89c132/156cc71e-604a-4062-8209-9f4827fd9816"
-					(reference "#PWR034")
+					(reference "#PWR033")
 					(unit 1)
 				)
@@
 		(dnp no)
 		(fields_autoplaced yes)
-		(property "Reference" "#PWR036"
+		(property "Reference" "#PWR035"
 			(at 86.36 133.35 0)
 			(effects
@@
 			(project "BLDC_driver"
 				(path "/6f399879-dc45-4210-87b6-ea005f89c132/156cc71e-604a-4062-8209-9f4827fd9816"
-					(reference "#PWR036")
+					(reference "#PWR035")
 					(unit 1)
 				)
@@
 		(on_board yes)
 		(dnp no)
-		(property "Reference" "#PWR030"
+		(property "Reference" "#PWR029"
 			(at 187.96 93.98 0)
 			(effects
@@
 			(project "BLDC_driver"
 				(path "/6f399879-dc45-4210-87b6-ea005f89c132/156cc71e-604a-4062-8209-9f4827fd9816"
-					(reference "#PWR030")
+					(reference "#PWR029")
 					(unit 1)
 				)
@@
 		(on_board yes)
 		(dnp no)
-		(property "Reference" "C15"
+		(property "Reference" "C19"
 			(at 76.708 123.19 0)
 			(effects
@@
 			(project "BLDC_driver"
 				(path "/6f399879-dc45-4210-87b6-ea005f89c132/156cc71e-604a-4062-8209-9f4827fd9816"
-					(reference "C15")
+					(reference "C19")
 					(unit 1)
 				)
@@
 		(dnp no)
 		(fields_autoplaced yes)
-		(property "Reference" "#PWR039"
+		(property "Reference" "#PWR038"
 			(at 86.36 153.67 0)
 			(effects
@@
 			(project "BLDC_driver"
 				(path "/6f399879-dc45-4210-87b6-ea005f89c132/156cc71e-604a-4062-8209-9f4827fd9816"
-					(reference "#PWR039")
+					(reference "#PWR038")
 					(unit 1)
 				)
@@
 		(on_board yes)
 		(dnp no)
-		(property "Reference" "#PWR041"
+		(property "Reference" "#PWR040"
 			(at 45.72 163.83 0)
 			(effects
@@
 			(project "BLDC_driver"
 				(path "/6f399879-dc45-4210-87b6-ea005f89c132/156cc71e-604a-4062-8209-9f4827fd9816"
-					(reference "#PWR041")
+					(reference "#PWR040")
 					(unit 1)
 				)
@@
 		(on_board yes)
 		(dnp no)
-		(property "Reference" "#PWR028"
+		(property "Reference" "#PWR027"
 			(at 74.93 45.085 0)
 			(effects
@@
 			(project "BLDC_driver"
 				(path "/6f399879-dc45-4210-87b6-ea005f89c132/156cc71e-604a-4062-8209-9f4827fd9816"
-					(reference "#PWR028")
+					(reference "#PWR027")
 					(unit 1)
 				)
@@
 		(on_board yes)
 		(dnp no)
-		(property "Reference" "#PWR035"
+		(property "Reference" "#PWR034"
 			(at 45.72 123.19 0)
 			(effects
@@
 			(project "BLDC_driver"
 				(path "/6f399879-dc45-4210-87b6-ea005f89c132/156cc71e-604a-4062-8209-9f4827fd9816"
-					(reference "#PWR035")
+					(reference "#PWR034")
 					(unit 1)
 				)
@@
 		(on_board yes)
 		(dnp no)
-		(property "Reference" "#PWR037"
+		(property "Reference" "#PWR036"
 			(at 45.72 134.62 0)
 			(effects
@@
 			(project "BLDC_driver"
 				(path "/6f399879-dc45-4210-87b6-ea005f89c132/156cc71e-604a-4062-8209-9f4827fd9816"
-					(reference "#PWR037")
+					(reference "#PWR036")
 					(unit 1)
 				)
@@
 		(on_board yes)
 		(dnp no)
-		(property "Reference" "C18"
+		(property "Reference" "C22"
 			(at 41.148 161.798 0)
 			(effects
@@
 			(project "BLDC_driver"
 				(path "/6f399879-dc45-4210-87b6-ea005f89c132/156cc71e-604a-4062-8209-9f4827fd9816"
-					(reference "C18")
+					(reference "C22")
 					(unit 1)
 				)
@@
 		(on_board yes)
 		(dnp no)
-		(property "Reference" "#PWR029"
+		(property "Reference" "#PWR028"
 			(at 156.21 93.98 0)
 			(effects
@@
 			(project "BLDC_driver"
 				(path "/6f399879-dc45-4210-87b6-ea005f89c132/156cc71e-604a-4062-8209-9f4827fd9816"
-					(reference "#PWR029")
+					(reference "#PWR028")
 					(unit 1)
 				)
@@
 		(on_board yes)
 		(dnp no)
-		(property "Reference" "#PWR032"
+		(property "Reference" "#PWR031"
 			(at 49.53 95.25 0)
 			(effects
@@
 			(project "BLDC_driver"
 				(path "/6f399879-dc45-4210-87b6-ea005f89c132/156cc71e-604a-4062-8209-9f4827fd9816"
-					(reference "#PWR032")
+					(reference "#PWR031")
 					(unit 1)
 				)
@@
 		(on_board yes)
 		(dnp no)
-		(property "Reference" "#PWR040"
+		(property "Reference" "#PWR039"
 			(at 45.72 154.94 0)
 			(effects
@@
 			(project "BLDC_driver"
 				(path "/6f399879-dc45-4210-87b6-ea005f89c132/156cc71e-604a-4062-8209-9f4827fd9816"
-					(reference "#PWR040")
+					(reference "#PWR039")
 					(unit 1)
 				)
@@
 		(on_board yes)
 		(dnp no)
-		(property "Reference" "C16"
+		(property "Reference" "C20"
 			(at 41.148 141.478 0)
 			(effects
@@
 			(project "BLDC_driver"
 				(path "/6f399879-dc45-4210-87b6-ea005f89c132/156cc71e-604a-4062-8209-9f4827fd9816"
-					(reference "C16")
+					(reference "C20")
 					(unit 1)
 				)
@@
 		(on_board yes)
 		(dnp no)
-		(property "Reference" "#PWR038"
+		(property "Reference" "#PWR037"
 			(at 45.72 143.51 0)
 			(effects
@@
 			(project "BLDC_driver"
 				(path "/6f399879-dc45-4210-87b6-ea005f89c132/156cc71e-604a-4062-8209-9f4827fd9816"
-					(reference "#PWR038")
+					(reference "#PWR037")
 					(unit 1)
 				)
@@
 		(on_board yes)
 		(dnp no)
-		(property "Reference" "C17"
+		(property "Reference" "C21"
 			(at 76.708 143.51 0)
 			(effects
@@
 			(project "BLDC_driver"
 				(path "/6f399879-dc45-4210-87b6-ea005f89c132/156cc71e-604a-4062-8209-9f4827fd9816"
-					(reference "C17")
+					(reference "C21")
 					(unit 1)
 				)
